File: Power Module/motor_controller.kicad_sch (KiCad schematic)
At the start: 22 parts, among them Q10 CSD18509Q5B, Q11 CSD18509Q5B, Q12 CSD18509Q5B, Q7 CSD18509Q5B, Q8 CSD18509Q5B, Q9 CSD18509Q5B, U3 MCF8329A1IREER

Commit message: wpi <<< mit
Parts:
- added J3: MOTOR, Custom:Edge_Solderpoint, symbol Connector:Conn_01x03_Pin
- C7: renamed from C17; footprint Capacitor_SMD:C_0603_1608Metric -> Capacitor_SMD:C_0402_1005Metric
- R13: renamed from R17; value R_SENSE -> 0.01; footprint Resistor_SMD:R_0402_1005Metric -> Resistor_SMD:R_2512_6332Metric
- renumbered C20 to C10, C21 to C11, C44 to C12, C22 to C13, C13 to C3, C14 to C4, C15 to C5, C16 to C6, C18 to C8, C19 to C9, Q7 to Q1, Q8 to Q2, Q9 to Q3, Q10 to Q4, Q11 to Q5, Q12 to Q6, R18 to R14, R19 to R15, R20 to R16, U3 to U2
Connections:
- net A: now also J3.1 (Pin_1)
- net B: now also J3.2 (Pin_2)
- net C: now also J3.3 (Pin_3)
- net GND: no longer Q2.1 (S), Q2.2 (S), Q2.3 (S), Q4.1 (S), Q4.2 (S), Q4.3 (S), Q6.1 (S), Q6.2 (S), Q6.3 (S), U2.21 (LSS)
- net +1V5: no longer names the net of C13.1, U2.36 (DVDD)
- net SN renamed LSS
- net LSS: now also Q2.1 (S), Q2.2 (S), Q2.3 (S), Q4.1 (S), Q4.2 (S), Q4.3 (S), Q6.1 (S), Q6.2 (S), Q6.3 (S), U2.21 (LSS)

Commit message: V1 design
Parts:
- renumbered J3 to J2
Changed lines of the file:
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@@
 		(dnp no)
 		(fields_autoplaced yes)
-		(property "Reference" "J3"
+		(property "Reference" "J2"
 			(at 212.09 146.0499 0)
 			(effects
