File: Power Module/Power Module.kicad_sch (KiCad schematic)
At the start: 24 parts, among them J1 ICC, J2 MOTOR 1, J3 MOTOR 3, J4 MOTOR 2, J5 MOTOR 4, U1 LM2576S-3.3

Commit message: wpi <<< mit
Parts:
- removed J1: ICC, Connector_PinHeader_2.54mm:PinHeader_2x12_P2.54mm_Vertical, symbol Connector_Generic:Conn_02x12_Counter_Clockwise
- removed J2: MOTOR 1, Custom:Edge_Solderpoint, symbol Connector:Conn_01x03_Pin
- removed J3: MOTOR 3, Custom:Edge_Solderpoint, symbol Connector:Conn_01x03_Pin
- removed J4: MOTOR 2, Custom:Edge_Solderpoint, symbol Connector:Conn_01x03_Pin
- removed J5: MOTOR 4, Custom:Edge_Solderpoint, symbol Connector:Conn_01x03_Pin
- added H1: MountingHole_Pad, MountingHole:MountingHole_3.2mm_M3_Pad, symbol Mechanical:MountingHole_Pad
- added J6: Conn_02x12_Odd_Even, Connector_PinHeader_2.54mm:PinHeader_2x12_P2.54mm_Vertical, symbol Connector_Generic:Conn_02x12_Odd_Even
Connections:
- net +3V3: now also J6.12 (Pin_12)
- net AGND: now also H1.1, J6.14 (Pin_14)
- net ENA_1: now also J6.3 (Pin_3)
- net ENA_2: now also J6.21 (Pin_21)
- net ENA_3: now also J6.15 (Pin_15)
- net ENA_4: now also J6.5 (Pin_5)
- net NFAULT_1: now also J6.6 (Pin_6)
- net NFAULT_2: now also J6.24 (Pin_24)
- net NFAULT_3: now also J6.18 (Pin_18)
- net NFAULT_4: now also J6.10 (Pin_10)
- net PWM_1: now also J6.1 (Pin_1)
- net PWM_2: now also J6.23 (Pin_23)
- net PWM_3: now also J6.17 (Pin_17)
- net PWM_4: now also J6.7 (Pin_7)
- net SCL: now also J6.11 (Pin_11)
- net SDA: now also J6.13 (Pin_13)
- net SPEED_1: now also J6.2 (Pin_2)
- net SPEED_2: now also J6.20 (Pin_20)
- net SPEED_3: now also J6.19 (Pin_19)
- net SPEED_4: now also J6.9 (Pin_9)
- net S_OX_1: now also J6.4 (Pin_4)
- net S_OX_2: now also J6.22 (Pin_22)
- net S_OX_3: now also J6.16 (Pin_16)
- net S_OX_4: now also J6.8 (Pin_8)
- no-connect marks 4 -> 0
Other:
- sheet Motor controller1 ports: added none; removed A, AVDD, B, C
- sheet Motor controller2 ports: added none; removed A, AVDD, B, C
- sheet Motor controller3 ports: added none; removed A, AVDD, B, C
- sheet Motor controller4 ports: added none; removed A, AVDD, B, C

Commit message: V1 design
Parts:
- removed C1: 100uF, Capacitor_SMD:C_0603_1608Metric, symbol Device:C
- removed C2: 1000uF, Capacitor_SMD:C_0603_1608Metric, symbol Device:C
- removed J6: Conn_02x12_Odd_Even, Connector_PinHeader_2.54mm:PinHeader_2x12_P2.54mm_Vertical, symbol Connector_Generic:Conn_02x12_Odd_Even
- added C1: 1000uF, Capacitor_Tantalum_SMD:CP_EIA-7343-30_AVX-N, symbol Device:C_Polarized
- added C47: 100uF, Capacitor_Tantalum_SMD:CP_EIA-7343-43_Kemet-X, symbol Device:C_Polarized
- added J1: Conn_02x14_Odd_Even, Connector_PinHeader_2.54mm:PinHeader_2x14_P2.54mm_Vertical, symbol Connector_Generic:Conn_02x14_Odd_Even
- added R29, R30, R31, R32: 4.7k, Resistor_SMD:R_0402_1005Metric, symbol Device:R
- added U6: TCA9548APWR, Package_SO:TSSOP-24_4.4x7.8mm_P0.65mm, symbol Interface_Expansion:TCA9548APWR
- R10, R3, R4, R9: value 0 -> 4.7k; footprint Resistor_SMD:R_0603_1608Metric_Pad0.98x0.95mm_HandSolder -> Resistor_SMD:R_0402_1005Metric
Connections:
- net +3V3: now also R10.1, R3.1, R4.1, R9.1, C1.1, J1.14 (Pin_14), R29.2, R30.2, R31.2, R32.2, U6.24 (VCC)
- net +BATT: now also C47.1, J1.1 (Pin_1), J1.2 (Pin_2)
- net AGND: now also C1.2, C47.2, J1.16 (Pin_16), J1.27 (Pin_27), J1.28 (Pin_28), U6.1 (A0), U6.12 (GND), U6.2 (A1), U6.21 (A2), U6.3 (~{RESET})
- net ENA_1: now also J1.5 (Pin_5)
- net ENA_2: now also J1.23 (Pin_23)
- net ENA_3: now also J1.17 (Pin_17)
- net ENA_4: now also J1.7 (Pin_7)
- net NFAULT_1: now also J1.8 (Pin_8)
- net NFAULT_2: now also J1.26 (Pin_26)
- net NFAULT_3: now also J1.20 (Pin_20)
- net NFAULT_4: now also J1.12 (Pin_12)
- net PWM_1: now also J1.3 (Pin_3)
- net PWM_2: now also J1.25 (Pin_25)
- net PWM_3: now also J1.19 (Pin_19)
- net PWM_4: now also J1.9 (Pin_9)
- net SCL: now also J1.15 (Pin_15), U6.22 (SCL)
- net SDA: now also J1.13 (Pin_13), U6.23 (SDA); no longer R10.1, R3.1, R4.1, R9.1
- net SPEED_1: now also J1.4 (Pin_4)
- net SPEED_2: now also J1.22 (Pin_22)
- net SPEED_3: now also J1.21 (Pin_21)
- net SPEED_4: now also J1.11 (Pin_11)
- net S_OX_1: now also J1.6 (Pin_6)
- net S_OX_2: now also J1.24 (Pin_24)
- net S_OX_3: now also J1.18 (Pin_18)
- net S_OX_4: now also J1.10 (Pin_10)
- net Motor controller1/SDA renamed SCL_1
- net SCL_1: now also U6.5 (SC0)
- net Motor controller2/SDA renamed SCL_2
- net SCL_2: now also U6.7 (SC1)
- net Motor controller3/SDA renamed SDA_1
- net SDA_1: now also U6.4 (SD0)
- net Motor controller4/SDA renamed SDA_2
- net SDA_2: now also U6.6 (SD1)
- new net SCL_3: R29.1, U6.9 (SC2)
- new net SCL_4: R31.1, U6.11 (SC3)
- new net SDA_3: R30.1, U6.8 (SD2)
- new net SDA_4: R32.1, U6.10 (SD3)
- no-connect marks 0 -> 8

Commit message: doofus, also added I2C multiplexer stuff
Parts:
- added R33: 4.7k, Resistor_SMD:R_0402_1005Metric, symbol Device:R
Connections:
- net +3V3: now also R33.1
- net AGND: no longer U6.3 (~{RESET})
- new net: R33.2, U6.3 (~{RESET})
Changed lines of the file:
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@@
-	)
-	(junction
-		(at 45.72 116.84)
-		(diameter 0)
-		(color 0 0 0 0)
 	)
 	(junction
@@
 	(wire
 		(pts
+			(xy 31.75 101.6) (xy 31.75 104.14)
+		)
+		(stroke
+			(width 0)
+			(type default)
+		)
+	)
+	(wire
+		(pts
 			(xy 231.14 39.37) (xy 233.68 39.37)
 		)
@@
 	(wire
 		(pts
+			(xy 31.75 104.14) (xy 36.83 104.14)
+		)
+		(stroke
+			(width 0)
+			(type default)
+		)
+	)
+	(wire
+		(pts
 			(xy 85.09 119.38) (xy 85.09 121.92)
 		)
@@
 	(wire
 		(pts
+			(xy 44.45 104.14) (xy 48.26 104.14)
+		)
+		(stroke
+			(width 0)
+			(type default)
+		)
+	)
+	(wire
+		(pts
 			(xy 143.51 143.51) (xy 140.97 143.51)
 		)
@@
 	(wire
 		(pts
-			(xy 45.72 104.14) (xy 45.72 116.84)
-		)
-		(stroke
-			(width 0)
-			(type default)
-		)
-	)
-	(wire
-		(pts
 			(xy 125.73 163.83) (xy 128.27 163.83)
 		)
@@
 		(pts
 			(xy 125.73 151.13) (xy 128.27 151.13)
-		)
-		(stroke
-			(width 0)
-			(type default)
-		)
-	)
-	(wire
-		(pts
-			(xy 48.26 104.14) (xy 45.72 104.14)
 		)
 		(stroke
@@
 	)
 	(symbol
+		(lib_id "power:+3V3")
+		(at 31.75 101.6 0)
+		(unit 1)
+		(exclude_from_sim no)
+		(in_bom yes)
+		(on_board yes)
+		(dnp no)
+		(fields_autoplaced yes)
+		(property "Reference" "#PWR093"
+			(at 31.75 105.41 0)
+			(effects
+				(font
+					(size 1.27 1.27)
+				)
+				(hide yes)
+			)
+		)
+		(property "Value" "+3V3"
+			(at 31.75 96.52 0)
+			(effects
+				(font
+					(size 1.27 1.27)
+				)
+			)
+		)
+		(property "Footprint" ""
+			(at 31.75 101.6 0)
+			(effects
+				(font
+					(size 1.27 1.27)
+				)
+				(hide yes)
+			)
+		)
+		(property "Datasheet" ""
+			(at 31.75 101.6 0)
+			(effects
+				(font
+					(size 1.27 1.27)
+				)
+				(hide yes)
+			)
+		)
+		(property "Description" "Power symbol creates a global label with name \"+3V3\""
+			(at 31.75 101.6 0)
+			(effects
+				(font
+					(size 1.27 1.27)
+				)
+				(hide yes)
+			)
+		)
+		(pin "1"
+		)
+		(instances
+			(project ""
+				(path "/f976c425-4c5c-4311-bdab-a894678168a5"
+					(reference "#PWR093")
+					(unit 1)
+				)
+			)
+		)
+	)
+	(symbol
 		(lib_id "power:GND")
 		(at 114.3 45.72 0)
@@
 					(unit 1)
 				)
+			)
+		)
+	)
+	(symbol
+		(lib_id "Device:R")
+		(at 40.64 104.14 90)
+		(unit 1)
+		(exclude_from_sim no)
+		(in_bom yes)
+		(on_board yes)
+		(dnp no)
+		(fields_autoplaced yes)
+		(property "Reference" "R33"
+			(at 40.64 97.79 90)
+			(effects
+				(font
+					(size 1.27 1.27)
+				)
+			)
+		)
+		(property "Value" "4.7k"
+			(at 40.64 100.33 90)
+			(effects
+				(font
+					(size 1.27 1.27)
+				)
+			)
+		)
+		(property "Footprint" "Resistor_SMD:R_0402_1005Metric"
+			(at 40.64 105.918 90)
+			(effects
+				(font
+					(size 1.27 1.27)
+				)
+				(hide yes)
+			)
+		)
+		(property "Datasheet" "~"
+			(at 40.64 104.14 0)
+			(effects
+				(font
+					(size 1.27 1.27)
+				)
+				(hide yes)
+			)
+		)
+		(property "Description" "Resistor"
+			(at 40.64 104.14 0)
+			(effects
+				(font
+					(size 1.27 1.27)
+				)
+				(hide yes)
+			)
+		)
+		(pin "2"
+		)
+		(pin "1"
+		)
+		(instances
+			(project ""
+				(path "/f976c425-4c5c-4311-bdab-a894678168a5"
+					(reference "R33")
+					(unit 1)
+				)
