File: Power Module/Power Module.kicad_pcb (KiCad board)
At the start: 2 copper layers, 94 x 94.5 mm, 112 parts, among them J1 ICC, J2 MOTOR 1, J3 MOTOR 3, J4 MOTOR 2, J5 MOTOR 4, Q1 CSD18509Q5B, Q10 CSD18509Q5B, Q11 CSD18509Q5B, Q12 CSD18509Q5B, Q13 CSD18509Q5B, Q14 CSD18509Q5B, Q15 CSD18509Q5B, Q16 CSD18509Q5B, Q17 CSD18509Q5B, Q18 CSD18509Q5B, Q19 CSD18509Q5B, Q2 CSD18509Q5B, Q20 CSD18509Q5B, Q21 CSD18509Q5B, Q22 CSD18509Q5B, Q23 CSD18509Q5B, Q24 CSD18509Q5B, Q3 CSD18509Q5B, Q4 CSD18509Q5B, Q5 CSD18509Q5B, Q6 CSD18509Q5B, Q7 CSD18509Q5B, Q8 CSD18509Q5B, Q9 CSD18509Q5B, U1 LM2576S-3.3, U2 MCF8329A1IREER, U3 MCF8329A1IREER, U4 MCF8329A1IREER, U5 MCF8329A1IREER

Commit message: wpi <<< mit
Parts:
- removed J1: ICC, Connector_PinHeader_2.54mm:PinHeader_2x12_P2.54mm_Vertical
- added H1: MountingHole_Pad, MountingHole:MountingHole_3.2mm_M3_Pad, F.Cu at (53.5, 48.7)
- added H1: MountingHole_Pad, MountingHole:MountingHole_3.2mm_M3_Pad, F.Cu at (128.5, 48.7)
- added H1: MountingHole_Pad, MountingHole:MountingHole_3.2mm_M3_Pad, F.Cu at (128.5, 113.7)
- added H1: MountingHole_Pad, MountingHole:MountingHole_3.2mm_M3_Pad, F.Cu at (53.5, 113.7)
- added J6: Conn_02x12_Odd_Even, Connector_PinHeader_2.54mm:PinHeader_2x12_P2.54mm_Vertical, F.Cu at (51.0, 67.2)
- C16, C26, C36: value 10uF -> 1uF; footprint Capacitor_SMD:C_0603_1608Metric -> Capacitor_SMD:C_0402_1005Metric
- C17: value 470nF -> 10uF; moved to F.Cu
- C18: value 47uF -> 470nF; footprint Capacitor_SMD:CP_Elec_6.3x7.7 -> Capacitor_SMD:C_0402_1005Metric
- C19: value 0.1uF -> 47uF; footprint Capacitor_SMD:C_0603_1608Metric -> Capacitor_SMD:CP_Elec_6.3x7.7
- C20, C42: value 1uF -> 0.1uF; footprint Capacitor_SMD:C_0402_1005Metric -> Capacitor_SMD:C_0603_1608Metric
- C21: value 470uF -> 1uF; footprint Capacitor_SMD:CP_Elec_10x10.5 -> Capacitor_SMD:C_0402_1005Metric
- C22, C33, C44: value 1uF -> 470uF; footprint Capacitor_SMD:C_0402_1005Metric -> Capacitor_SMD:CP_Elec_10x10.5
- C27, C37: value 470nF -> 1uF; footprint Capacitor_SMD:C_0603_1608Metric -> Capacitor_SMD:C_0402_1005Metric; moved to F.Cu
- C28: value 47uF -> 10uF; footprint Capacitor_SMD:CP_Elec_6.3x7.7 -> Capacitor_SMD:C_0603_1608Metric
- C29: value 0.1uF -> 470nF; footprint Capacitor_SMD:C_0603_1608Metric -> Capacitor_SMD:C_0402_1005Metric
- C30: value 1uF -> 47uF; footprint Capacitor_SMD:C_0402_1005Metric -> Capacitor_SMD:CP_Elec_6.3x7.7
- C31: value 470uF -> 0.1uF; footprint Capacitor_SMD:CP_Elec_10x10.5 -> Capacitor_SMD:C_0603_1608Metric
- C38: value 47uF -> 1uF; footprint Capacitor_SMD:CP_Elec_6.3x7.7 -> Capacitor_SMD:C_0402_1005Metric
- C39: value 0.1uF -> 10uF
- C40: value 1uF -> 470nF
- C41: value 470uF -> 47uF; footprint Capacitor_SMD:CP_Elec_10x10.5 -> Capacitor_SMD:CP_Elec_6.3x7.7
- C7: footprint Capacitor_SMD:C_0603_1608Metric -> Capacitor_SMD:C_0402_1005Metric; moved to F.Cu
- J2: value MOTOR 1 -> MOTOR
- J3: value MOTOR 3 -> MOTOR
- J4: value MOTOR 2 -> MOTOR
- J5: value MOTOR 4 -> MOTOR
- Q1, Q11, Q13, Q15, Q17, Q19, Q21, Q23, Q3, Q5, Q7, Q9: moved to F.Cu
- Q10, Q12, Q14, Q16, Q18, Q2, Q20, Q22, Q24, Q4, Q6, Q8, R1, R10, R11, R12, R2, R3, R4, R5, R6, R7, R8, R9: moved to B.Cu
- R13, R17, R21, R25: value R_SENSE -> 0.01; footprint Resistor_SMD:R_0402_1005Metric -> Resistor_SMD:R_2512_6332Metric; moved to B.Cu
- moved U1 175.6 mm to (-70.3, 100.9)
- moved D1 171.7 mm to (-59.2, 107.0)
- moved C2 164.4 mm to (-61.4, 92.3)
- moved L1 158.2 mm to (-56.1, 81.4), turned to 0 degrees
- moved D2 157.0 mm to (-57.4, 89.8)
- moved C1 156.7 mm to (-61.4, 89.8), turned to 0 degrees
- moved J4 92.6 mm to (112.5, 123.5), turned to 180 degrees
- moved J2 92.0 mm to (80.4, 123.5), turned to 180 degrees
- moved J5 90.8 mm to (101.6, 38.9), turned to 0 degrees
- moved J3 90.2 mm to (69.5, 38.9), turned to 0 degrees
- moved C44 77.4 mm to (117.8, 66.5), turned to 0 degrees
- moved BT1 72.1 mm to (166.8, 80.4)
- moved Q19 70.0 mm to (109.1, 54.0), turned to -90 degrees
- moved Q20 70.0 mm to (109.1, 54.0), turned to 90 degrees
- moved C28 64.7 mm to (107.0, 100.5), turned to 90 degrees
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Connections:
- C12 pad 1: +1V5 -> Net-(U2-AVDD)
- C13 pad 1: /Motor controller1/SHA -> Net-(U2-DVDD)
- C13 pad 2: /Motor controller1/BSTA -> AGND
- C14 pad 1: /Motor controller1/SHB -> /Motor controller1/A
- C14 pad 2: /Motor controller1/BSTB -> /Motor controller1/BSTA
- C15 pad 1: /Motor controller1/SHC -> /Motor controller1/B
- C15 pad 2: /Motor controller1/BSTC -> /Motor controller1/BSTB
- C16 pad 1: AGND -> /Motor controller1/C
- C16 pad 2: Net-(U3-GVDD) -> /Motor controller1/BSTC
- C17 pad 1: Net-(U3-CPH) -> AGND
- C17 pad 2: Net-(U3-CPL) -> Net-(U3-GVDD)
- C18 pad 1: +BATT -> Net-(U3-CPH)
- C18 pad 2: AGND -> Net-(U3-CPL)
- C19 pad 1: AGND -> +BATT
- C19 pad 2: +BATT -> AGND
- C20 pad 1: +3V3 -> AGND
- C20 pad 2: AGND -> +BATT
- C21 pad 1: +BATT -> +3V3
- C22 pad 1: +1V5 -> +BATT
- C23 pad 1: /Motor controller3/SHA -> Net-(U3-AVDD)
- C23 pad 2: /Motor controller3/BSTA -> AGND
- C24 pad 1: /Motor controller3/SHB -> Net-(U3-DVDD)
- C24 pad 2: /Motor controller3/BSTB -> AGND
- C25 pad 1: /Motor controller3/SHC -> /Motor controller3/A
- C25 pad 2: /Motor controller3/BSTC -> /Motor controller3/BSTA
- C26 pad 1: AGND -> /Motor controller3/B
- C26 pad 2: Net-(U4-GVDD) -> /Motor controller3/BSTB
- C27 pad 1: Net-(U4-CPH) -> /Motor controller3/C
- C27 pad 2: Net-(U4-CPL) -> /Motor controller3/BSTC
- C28 pad 1: +BATT -> AGND
- C28 pad 2: AGND -> Net-(U4-GVDD)
- C29 pad 1: AGND -> Net-(U4-CPH)
- C29 pad 2: +BATT -> Net-(U4-CPL)
- C3 pad 1: /Motor controller2/SHA -> /Motor controller2/A
- C30 pad 1: +3V3 -> +BATT
- C31 pad 1: +BATT -> AGND
- C31 pad 2: AGND -> +BATT
- C32 pad 1: +1V5 -> +3V3
- C33 pad 1: /Motor controller4/SHA -> +BATT
- C33 pad 2: /Motor controller4/BSTA -> AGND
- C34 pad 1: /Motor controller4/SHB -> Net-(U4-AVDD)
- C34 pad 2: /Motor controller4/BSTB -> AGND
- C35 pad 1: /Motor controller4/SHC -> Net-(U4-DVDD)
- C35 pad 2: /Motor controller4/BSTC -> AGND
- C36 pad 1: AGND -> /Motor controller4/A
- C36 pad 2: Net-(U5-GVDD) -> /Motor controller4/BSTA
- C37 pad 1: Net-(U5-CPH) -> /Motor controller4/B
- C37 pad 2: Net-(U5-CPL) -> /Motor controller4/BSTB
- C38 pad 1: +BATT -> /Motor controller4/C
- C38 pad 2: AGND -> /Motor controller4/BSTC
- C39 pad 2: +BATT -> Net-(U5-GVDD)
- C4 pad 1: /Motor controller2/SHB -> /Motor controller2/B
- C40 pad 1: +3V3 -> Net-(U5-CPH)
- C40 pad 2: AGND -> Net-(U5-CPL)
- C42 pad 1: +1V5 -> AGND
- C42 pad 2: AGND -> +BATT
- C43 pad 1: Net-(U2-AVDD) -> +3V3
- C44 pad 1: Net-(U3-AVDD) -> +BATT
- C45 pad 1: Net-(U4-AVDD) -> Net-(U5-AVDD)
- C46 pad 1: Net-(U5-AVDD) -> Net-(U5-DVDD)
- C5 pad 1: /Motor controller2/SHC -> /Motor controller2/C
- J2 pad 1: /Motor controller1/SHC -> /Motor controller2/A
- J2 pad 2: /Motor controller1/SHB -> /Motor controller2/B
- J2 pad 3: /Motor controller1/SHA -> /Motor controller2/C
- J3 pad 1: /Motor controller3/SHC -> /Motor controller1/A
- J3 pad 2: /Motor controller3/SHB -> /Motor controller1/B
- J3 pad 3: /Motor controller3/SHA -> /Motor controller1/C
- J4 pad 1: /Motor controller2/SHC -> /Motor controller3/A
- J4 pad 2: /Motor controller2/SHB -> /Motor controller3/B
- J4 pad 3: /Motor controller2/SHA -> /Motor controller3/C
- J5 pad 1: /Motor controller4/SHC -> /Motor controller4/A
- J5 pad 2: /Motor controller4/SHB -> /Motor controller4/B
- J5 pad 3: /Motor controller4/SHA -> /Motor controller4/C
- Q1 pad 1: /Motor controller2/SHA -> /Motor controller2/A
- Q1 pad 2: /Motor controller2/SHA -> /Motor controller2/A
- Q1 pad 3: /Motor controller2/SHA -> /Motor controller2/A
- Q10 pad 1: AGND -> /Motor controller1/LSS
- Q10 pad 2: AGND -> /Motor controller1/LSS
- Q10 pad 3: AGND -> /Motor controller1/LSS
- Q10 pad 5: /Motor controller1/SHB -> /Motor controller1/B
- Q11 pad 1: /Motor controller1/SHC -> /Motor controller1/C
- Q11 pad 2: /Motor controller1/SHC -> /Motor controller1/C
- Q11 pad 3: /Motor controller1/SHC -> /Motor controller1/C
- Q12 pad 1: AGND -> /Motor controller1/LSS
- Q12 pad 2: AGND -> /Motor controller1/LSS
- Q12 pad 3: AGND -> /Motor controller1/LSS
- Q12 pad 5: /Motor controller1/SHC -> /Motor controller1/C
- Q13 pad 1: /Motor controller3/SHA -> /Motor controller3/A
- Q13 pad 2: /Motor controller3/SHA -> /Motor controller3/A
- Q13 pad 3: /Motor controller3/SHA -> /Motor controller3/A
- Q14 pad 1: AGND -> /Motor controller3/LSS
- Q14 pad 2: AGND -> /Motor controller3/LSS
- Q14 pad 3: AGND -> /Motor controller3/LSS
- Q14 pad 5: /Motor controller3/SHA -> /Motor controller3/A
- Q15 pad 1: /Motor controller3/SHB -> /Motor controller3/B
- Q15 pad 2: /Motor controller3/SHB -> /Motor controller3/B
- Q15 pad 3: /Motor controller3/SHB -> /Motor controller3/B
- Q16 pad 1: AGND -> /Motor controller3/LSS
- Q16 pad 2: AGND -> /Motor controller3/LSS
- Q16 pad 3: AGND -> /Motor controller3/LSS
- Q16 pad 5: /Motor controller3/SHB -> /Motor controller3/B
- Q17 pad 1: /Motor controller3/SHC -> /Motor controller3/C
- Q17 pad 2: /Motor controller3/SHC -> /Motor controller3/C
- Q17 pad 3: /Motor controller3/SHC -> /Motor controller3/C
- Q18 pad 1: AGND -> /Motor controller3/LSS
- Q18 pad 2: AGND -> /Motor controller3/LSS
- Q18 pad 3: AGND -> /Motor controller3/LSS
- Q18 pad 5: /Motor controller3/SHC -> /Motor controller3/C
- Q19 pad 1: /Motor controller4/SHA -> /Motor controller4/A
- Q19 pad 2: /Motor controller4/SHA -> /Motor controller4/A
- Q19 pad 3: /Motor controller4/SHA -> /Motor controller4/A
- Q2 pad 1: AGND -> /Motor controller2/LSS
- Q2 pad 2: AGND -> /Motor controller2/LSS
- Q2 pad 3: AGND -> /Motor controller2/LSS
- Q2 pad 5: /Motor controller2/SHA -> /Motor controller2/A
- Q20 pad 1: AGND -> /Motor controller4/LSS
- Q20 pad 2: AGND -> /Motor controller4/LSS
- Q20 pad 3: AGND -> /Motor controller4/LSS
- Q20 pad 5: /Motor controller4/SHA -> /Motor controller4/A
- Q21 pad 1: /Motor controller4/SHB -> /Motor controller4/B
- Q21 pad 2: /Motor controller4/SHB -> /Motor controller4/B
- Q21 pad 3: /Motor controller4/SHB -> /Motor controller4/B
- Q22 pad 1: AGND -> /Motor controller4/LSS
- Q22 pad 2: AGND -> /Motor controller4/LSS
- Q22 pad 3: AGND -> /Motor controller4/LSS
- Q22 pad 5: /Motor controller4/SHB -> /Motor controller4/B
- Q23 pad 1: /Motor controller4/SHC -> /Motor controller4/C
- Q23 pad 2: /Motor controller4/SHC -> /Motor controller4/C
- Q23 pad 3: /Motor controller4/SHC -> /Motor controller4/C
- Q24 pad 1: AGND -> /Motor controller4/LSS
- Q24 pad 2: AGND -> /Motor controller4/LSS
- Q24 pad 3: AGND -> /Motor controller4/LSS
- Q24 pad 5: /Motor controller4/SHC -> /Motor controller4/C
- Q3 pad 1: /Motor controller2/SHB -> /Motor controller2/B
- Q3 pad 2: /Motor controller2/SHB -> /Motor controller2/B
- Q3 pad 3: /Motor controller2/SHB -> /Motor controller2/B
- Q4 pad 1: AGND -> /Motor controller2/LSS
- Q4 pad 2: AGND -> /Motor controller2/LSS
- Q4 pad 3: AGND -> /Motor controller2/LSS
- Q4 pad 5: /Motor controller2/SHB -> /Motor controller2/B
- Q5 pad 1: /Motor controller2/SHC -> /Motor controller2/C
- Q5 pad 2: /Motor controller2/SHC -> /Motor controller2/C
- Q5 pad 3: /Motor controller2/SHC -> /Motor controller2/C
- Q6 pad 1: AGND -> /Motor controller2/LSS
- Q6 pad 2: AGND -> /Motor controller2/LSS
- Q6 pad 3: AGND -> /Motor controller2/LSS
- Q6 pad 5: /Motor controller2/SHC -> /Motor controller2/C
- Q7 pad 1: /Motor controller1/SHA -> /Motor controller1/A
- Q7 pad 2: /Motor controller1/SHA -> /Motor controller1/A
- Q7 pad 3: /Motor controller1/SHA -> /Motor controller1/A
- Q8 pad 1: AGND -> /Motor controller1/LSS
- Q8 pad 2: AGND -> /Motor controller1/LSS
- Q8 pad 3: AGND -> /Motor controller1/LSS
- Q8 pad 5: /Motor controller1/SHA -> /Motor controller1/A
- Q9 pad 1: /Motor controller1/SHB -> /Motor controller1/B
- Q9 pad 2: /Motor controller1/SHB -> /Motor controller1/B
- Q9 pad 3: /Motor controller1/SHB -> /Motor controller1/B
- R13 pad 1: /Motor controller2/SN -> /Motor controller2/LSS
- R17 pad 1: /Motor controller1/SN -> /Motor controller1/LSS
- R21 pad 1: /Motor controller3/SN -> /Motor controller3/LSS
- R25 pad 1: /Motor controller4/SN -> /Motor controller4/LSS
- U2 pad 10: /Motor controller2/SHA -> /Motor controller2/A
- U2 pad 14: /Motor controller2/SHB -> /Motor controller2/B
- U2 pad 18: /Motor controller2/SHC -> /Motor controller2/C
- U2 pad 21: AGND -> /Motor controller2/LSS
- U2 pad 23: /Motor controller2/SN -> /Motor controller2/LSS
- U2 pad 36: +1V5 -> Net-(U2-DVDD)
- U3 pad 10: /Motor controller1/SHA -> /Motor controller1/A
- U3 pad 14: /Motor controller1/SHB -> /Motor controller1/B
- U3 pad 18: /Motor controller1/SHC -> /Motor controller1/C
- U3 pad 21: AGND -> /Motor controller1/LSS
- U3 pad 23: /Motor controller1/SN -> /Motor controller1/LSS
- U3 pad 36: +1V5 -> Net-(U3-DVDD)
- U4 pad 10: /Motor controller3/SHA -> /Motor controller3/A
- U4 pad 14: /Motor controller3/SHB -> /Motor controller3/B
- U4 pad 18: /Motor controller3/SHC -> /Motor controller3/C
- U4 pad 21: AGND -> /Motor controller3/LSS
- U4 pad 23: /Motor controller3/SN -> /Motor controller3/LSS
- U4 pad 36: +1V5 -> Net-(U4-DVDD)
- U5 pad 10: /Motor controller4/SHA -> /Motor controller4/A
- U5 pad 14: /Motor controller4/SHB -> /Motor controller4/B
- U5 pad 18: /Motor controller4/SHC -> /Motor controller4/C
- U5 pad 21: AGND -> /Motor controller4/LSS
- U5 pad 23: /Motor controller4/SN -> /Motor controller4/LSS
- U5 pad 36: +1V5 -> Net-(U5-DVDD)
Routing:
- net +3V3: track 237.0 -> 32.6 mm, vias 16 -> 0
- net /ENA_3: track 24.3 -> 83.0 mm, vias 2 -> 1
- net /PWM_3: track 24.5 -> 81.4 mm
- net /SPEED_3: track 25.3 -> 77.6 mm, vias 1 -> 0
- net /S_OX_3: track 20.4 -> 68.4 mm, vias 0 -> 2
- net /NFAULT_3: track 24.1 -> 66.2 mm
- net AGND: track 87.1 -> 54.6 mm, vias 8 -> 68
- net /NFAULT_4: track 26.0 -> 57.3 mm
- net Net-(D1-K): track 28.8 -> 0.00 mm
- net /SCL: track 130.5 -> 157.6 mm, vias 5 -> 8
- net /SDA: track 109.9 -> 136.0 mm, vias 6 -> 8
- net /PWM_2: track 24.1 -> 49.4 mm
- net /ENA_2: track 29.4 -> 53.1 mm, vias 2 -> 0
- net /S_OX_4: track 34.6 -> 55.3 mm
- net /SPEED_4: track 39.6 -> 59.3 mm
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- added copper zone on F.Cu, net +BATT
- added copper zone on B.Cu, net /Motor controller1/A
- added copper zone on F.Cu, net /Motor controller1/A
- added copper zone on B.Cu, net /Motor controller1/B
- added copper zone on F.Cu, net /Motor controller1/B
- added copper zone on B.Cu, net /Motor controller1/C
- added copper zone on F.Cu, net /Motor controller1/C
- added copper zone on B.Cu, net /Motor controller1/LSS
- added copper zone on B.Cu, net /Motor controller2/A
- added copper zone on F.Cu, net /Motor controller2/A
- added copper zone on B.Cu, net /Motor controller2/B
- added copper zone on F.Cu, net /Motor controller2/B
- added copper zone on B.Cu, net /Motor controller2/C
- added copper zone on F.Cu, net /Motor controller2/C
- added copper zone on B.Cu, net /Motor controller2/LSS
- added copper zone on B.Cu, net /Motor controller3/A
- added copper zone on F.Cu, net /Motor controller3/A
- added copper zone on B.Cu, net /Motor controller3/B
- added copper zone on F.Cu, net /Motor controller3/B
- added copper zone on B.Cu, net /Motor controller3/C
- added copper zone on F.Cu, net /Motor controller3/C
- added copper zone on B.Cu, net /Motor controller3/LSS
- added copper zone on B.Cu, net /Motor controller4/A
- added copper zone on F.Cu, net /Motor controller4/A
- added copper zone on B.Cu, net /Motor controller4/B
- added copper zone on F.Cu, net /Motor controller4/B
- added copper zone on B.Cu, net /Motor controller4/C
- added copper zone on F.Cu, net /Motor controller4/C
- added copper zone on B.Cu, net /Motor controller4/LSS
- removed copper zone on B.Cu, net +BATT
- removed copper zone on B.Cu, net /Motor controller1/SHA
- removed copper zone on F.Cu, net /Motor controller1/SHA
- removed copper zone on B.Cu, net /Motor controller1/SHB
- removed copper zone on F.Cu, net /Motor controller1/SHB
- removed copper zone on B.Cu, net /Motor controller1/SHC
- removed copper zone on F.Cu, net /Motor controller1/SHC
- removed copper zone on B.Cu, net /Motor controller2/SHA
- removed copper zone on F.Cu, net /Motor controller2/SHA
- removed copper zone on B.Cu, net /Motor controller2/SHB
- removed copper zone on F.Cu, net /Motor controller2/SHB
- removed copper zone on B.Cu, net /Motor controller2/SHC
- removed copper zone on F.Cu, net /Motor controller2/SHC
- removed copper zone on B.Cu, net /Motor controller3/SHA
- removed copper zone on F.Cu, net /Motor controller3/SHA
- removed copper zone on B.Cu, net /Motor controller3/SHB
- removed copper zone on F.Cu, net /Motor controller3/SHB
- removed copper zone on B.Cu, net /Motor controller3/SHC
- removed copper zone on F.Cu, net /Motor controller3/SHC
- removed copper zone on B.Cu, net /Motor controller4/SHA
- removed copper zone on F.Cu, net /Motor controller4/SHA
- removed copper zone on B.Cu, net /Motor controller4/SHB
- removed copper zone on F.Cu, net /Motor controller4/SHB
- removed copper zone on B.Cu, net /Motor controller4/SHC
- removed copper zone on F.Cu, net /Motor controller4/SHC
- removed copper zone on F.Cu, net AGND
Other:
- board outline removed
- board text removed: "Your Brazilian Rainforest:tm delivery drone"

Commit message: 0 DRC errors wooooo
Parts:
- C1, C2, D1, U1: moved to B.Cu
- moved U1 201.5 mm to (131.2, 103.1), turned to -90 degrees
- moved C2 189.1 mm to (127.5, 83.5), turned to 90 degrees
- moved L1 188.1 mm to (131.6, 68.0), turned to -90 degrees
- moved C1 185.9 mm to (124.5, 90.5), turned to 90 degrees
- moved D1 183.1 mm to (123.5, 95.5), turned to 90 degrees
- moved D2 172.3 mm to (114.5, 78.0), turned to 180 degrees
- moved BT1 45.5 mm to (121.3, 79.9)
Routing:
- net +3V3: track 32.6 -> 283.0 mm, vias 0 -> 19
- net +BATT: track 55.9 -> 143.3 mm, vias 0 -> 1
- net Net-(D1-K): track 0.00 -> 48.2 mm, vias 0 -> 1
- net AGND: track 54.6 -> 92.3 mm, vias 68 -> 84
- net /SDA: track 136.0 -> 138.2 mm, vias 8 -> 9
- net /S_OX_2: track 35.1 -> 36.0 mm
- net /SPEED_3: track 77.6 -> 78.5 mm
- added copper zone on B.Cu, net AGND
Other:
- board outline added: 89.2 x 84.8 mm
- board text added: "3V3"
- board text added: "GND"
- board text added: "SDA"

Commit message: V1 design
Parts:
- removed J6: Conn_02x12_Odd_Even, Connector_PinHeader_2.54mm:PinHeader_2x12_P2.54mm_Vertical
- added C47: 100uF, Capacitor_Tantalum_SMD:CP_EIA-7343-43_Kemet-X, F.Cu at (128.0, 99.0)
- added J1: Conn_02x14_Odd_Even, Connector_PinHeader_2.54mm:PinHeader_2x14_P2.54mm_Vertical, F.Cu at (51.0, 64.7)
- added R29: 4.7k, Resistor_SMD:R_0402_1005Metric, F.Cu at (88.5, 86.0)
- added R30: 4.7k, Resistor_SMD:R_0402_1005Metric, F.Cu at (89.5, 81.0)
- added R31: 4.7k, Resistor_SMD:R_0402_1005Metric, F.Cu at (92.0, 75.5)
- added R32: 4.7k, Resistor_SMD:R_0402_1005Metric, F.Cu at (89.5, 75.5)
- added U6: TCA9548APWR, Package_SO:TSSOP-24_4.4x7.8mm_P0.65mm, B.Cu at (82.1, 81.4)
- C1: value 100uF -> 1000uF; footprint Capacitor_SMD:C_0603_1608Metric -> Capacitor_Tantalum_SMD:CP_EIA-7343-30_AVX-N; moved to F.Cu
- R10, R3, R4, R9: value 0 -> 4.7k; footprint Resistor_SMD:R_0603_1608Metric_Pad0.98x0.95mm_HandSolder -> Resistor_SMD:R_0402_1005Metric; moved to F.Cu
- moved R4 40.4 mm to (79.0, 76.0), turned to 0 degrees
- moved R3 14.9 mm to (76.5, 80.5), turned to -90 degrees
- moved R10 13.0 mm to (91.5, 81.0), turned to 180 degrees
- moved C1 12.0 mm to (133.0, 99.0), turned to -90 degrees
- moved R9 4.09 mm to (86.0, 89.0), turned to 180 degrees
Connections:
- C1 pad 1: +BATT -> +3V3
- R10 pad 1: /SDA -> +3V3
- R10 pad 2: /Motor controller4/SDA -> /SDA_2
- R3 pad 1: /SDA -> +3V3
- R3 pad 2: /Motor controller1/SDA -> /SCL_1
- R4 pad 1: /SDA -> +3V3
- R4 pad 2: /Motor controller3/SDA -> /SDA_1
- R9 pad 1: /SDA -> +3V3
- R9 pad 2: /Motor controller2/SDA -> /SCL_2
- U2 pad 29: /Motor controller2/SDA -> /SDA_2
- U2 pad 30: /SCL -> /SCL_2
- U3 pad 29: /Motor controller1/SDA -> /SDA_1
- U3 pad 30: /SCL -> /SCL_1
- U4 pad 29: /Motor controller3/SDA -> /SDA_3
- U4 pad 30: /SCL -> /SCL_3
- U5 pad 29: /Motor controller4/SDA -> /SDA_4
- U5 pad 30: /SCL -> /SCL_4
Routing:
- net /SCL: track 157.6 -> 32.6 mm, vias 8 -> 2
- net /SDA: track 138.2 -> 33.2 mm, vias 9 -> 1
- net /SDA_3: track 0.00 -> 45.3 mm, vias 0 -> 3
- net /SCL_3: track 0.00 -> 43.5 mm, vias 0 -> 3
- net /SCL_1: track 0.00 -> 33.8 mm, vias 0 -> 5
- net /SDA_2: track 0.00 -> 29.2 mm, vias 0 -> 5
- net /SCL_2: track 0.00 -> 25.8 mm, vias 0 -> 5
- net /SCL_4: track 0.00 -> 24.8 mm, vias 0 -> 3
- net /SDA_1: track 0.00 -> 23.6 mm, vias 0 -> 3
- net /SDA_4: track 0.00 -> 23.4 mm, vias 0 -> 1
- net +3V3: track 283.0 -> 305.0 mm, vias 19 -> 24
- net +BATT: track 143.3 -> 162.3 mm, vias 1 -> 3
- net /Motor controller1/SDA: track 3.83 -> 0.00 mm, vias 1 -> 0
- net /Motor controller3/SDA: track 3.83 -> 0.00 mm, vias 1 -> 0
- net /Motor controller4/SDA: track 3.83 -> 0.00 mm, vias 1 -> 0
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Other:
- outline, holes or cut-outs redrawn
- board text added: "Cardinal Power V1"
- board text removed: "SDA"

Commit message: doofus, also added I2C multiplexer stuff
Parts:
- added R33: 4.7k, Resistor_SMD:R_0402_1005Metric, B.Cu at (76.0, 81.0)
Connections:
- U6 pad 3: AGND -> Net-(U6-~{RESET})
Routing:
- net Net-(U6-~{RESET}): track 0.00 -> 4.80 mm
- net +3V3: track 305.0 -> 306.5 mm, vias 24 -> 25

Commit message: More localization work
Parts:
- removed C2: 1000uF, Capacitor_SMD:C_0603_1608Metric
Routing:
- net +3V3: track 306.5 -> 304.4 mm
Changed lines of the file:
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@@
 		(tags "resistor")
 		(property "Reference" "R33"
-			(at 0 1.17 360)
+			(at 0 1.17 0)
 			(layer "B.SilkS")
 			(effects
@@
 		)
 		(property "Value" "4.7k"
-			(at 0 -1.17 360)
+			(at 0 -1.17 0)
 			(layer "B.Fab")
 			(effects
@@
 		)
 		(fp_text user "${REFERENCE}"
-			(at 0 0 360)
+			(at 0 0 0)
 			(layer "B.Fab")
 			(effects
@@
 		)
 	)
-	(footprint "Capacitor_SMD:C_0603_1608Metric"
-		(layer "B.Cu")
-		(at 127.5 83.5 90)
-		(descr "Capacitor SMD 0603 (1608 Metric), square (rectangular) end terminal, IPC_7351 nominal, (Body size source: IPC-SM-782 page 76, https://www.pcb-3d.com/wordpress/wp-content/uploads/ipc-sm-782a_amendment_1_and_2.pdf), generated with kicad-footprint-generator")
-		(tags "capacitor")
-		(property "Reference" "C2"
-			(at 0 1.43 90)
-			(layer "B.SilkS")
-			(effects
-				(font
-					(size 1 1)
-					(thickness 0.15)
-				)
-				(justify mirror)
-			)
-		)
-		(property "Value" "1000uF"
-			(at 0 -1.43 90)
-			(layer "B.Fab")
-			(effects
-				(font
-					(size 1 1)
-					(thickness 0.15)
-				)
-				(justify mirror)
-			)
-		)
-		(property "Footprint" "Capacitor_SMD:C_0603_1608Metric"
-			(at 0 0 -90)
-			(unlocked yes)
-			(layer "B.Fab")
-			(hide yes)
-			(effects
-				(font
-					(size 1.27 1.27)
-					(thickness 0.15)
-				)
-				(justify mirror)
-			)
-		)
-		(property "Datasheet" ""
-			(at 0 0 -90)
-			(unlocked yes)
-			(layer "B.Fab")
-			(hide yes)
-			(effects
-				(font
-					(size 1.27 1.27)
-					(thickness 0.15)
-				)
-				(justify mirror)
-			)
-		)
-		(property "Description" "Unpolarized capacitor"
-			(at 0 0 -90)
-			(unlocked yes)
-			(layer "B.Fab")
-			(hide yes)
-			(effects
-				(font
-					(size 1.27 1.27)
-					(thickness 0.15)
-				)
-				(justify mirror)
-			)
-		)
-		(property ki_fp_filters "C_*")
-		(sheetname "Root")
-		(sheetfile "Power Module.kicad_sch")
-		(attr smd)
-		(fp_line
-			(start 0.14058 -0.51)
-			(end -0.14058 -0.51)
-			(stroke
-				(width 0.12)
-				(type solid)
-			)
-			(layer "B.SilkS")
-		)
-		(fp_line
-			(start 0.14058 0.51)
-			(end -0.14058 0.51)
-			(stroke
-				(width 0.12)
-				(type solid)
-			)
-			(layer "B.SilkS")
-		)
-		(fp_line
-			(start 1.48 -0.73)
-			(end 1.48 0.73)
-			(stroke
-				(width 0.05)
-				(type solid)
-			)
-			(layer "B.CrtYd")
-		)
-		(fp_line
-			(start -1.48 -0.73)
-			(end 1.48 -0.73)
-			(stroke
-				(width 0.05)
-				(type solid)
-			)
-			(layer "B.CrtYd")
-		)
-		(fp_line
-			(start 1.48 0.73)
-			(end -1.48 0.73)
-			(stroke
-				(width 0.05)
-				(type solid)
-			)
-			(layer "B.CrtYd")
-		)
-		(fp_line
-			(start -1.48 0.73)
-			(end -1.48 -0.73)
-			(stroke
-				(width 0.05)
-				(type solid)
-			)
-			(layer "B.CrtYd")
-		)
-		(fp_line
-			(start 0.8 -0.4)
-			(end 0.8 0.4)
-			(stroke
-				(width 0.1)
-				(type solid)
-			)
-			(layer "B.Fab")
-		)
-		(fp_line
-			(start -0.8 -0.4)
-			(end 0.8 -0.4)
-			(stroke
-				(width 0.1)
-				(type solid)
-			)
-			(layer "B.Fab")
-		)
-		(fp_line
-			(start 0.8 0.4)
-			(end -0.8 0.4)
-			(stroke
-				(width 0.1)
-				(type solid)
-			)
-			(layer "B.Fab")
-		)
-		(fp_line
-			(start -0.8 0.4)
-			(end -0.8 -0.4)
-			(stroke
-				(width 0.1)
-				(type solid)
-			)
-			(layer "B.Fab")
-		)
-		(fp_text user "${REFERENCE}"
-			(at 0 0 90)
-			(layer "B.Fab")
-			(effects
-				(font
-					(size 0.4 0.4)
-					(thickness 0.06)
-				)
-				(justify mirror)
-			)
-		)
-		(pad "1" smd roundrect
-			(at -0.775 0 90)
-			(size 0.9 0.95)
-			(layers "B.Cu" "B.Paste" "B.Mask")
-			(roundrect_rratio 0.25)
-			(net 3 "+3V3")
-			(pintype "passive")
-		)
-		(pad "2" smd roundrect
-			(at 0.775 0 90)
-			(size 0.9 0.95)
-			(layers "B.Cu" "B.Paste" "B.Mask")
-			(roundrect_rratio 0.25)
-			(net 2 "AGND")
-			(pintype "passive")
-		)
-		(model "${KICAD8_3DMODEL_DIR}/Capacitor_SMD.3dshapes/C_0603_1608Metric.wrl"
-			(offset
-				(xyz 0 0 0)
-			)
-			(scale
-				(xyz 1 1 1)
-			)
-			(rotate
-				(xyz 0 0 0)
-			)
-		)
-	)
 	(footprint "Resistor_SMD:R_0603_1608Metric_Pad0.98x0.95mm_HandSolder"
 		(layer "B.Cu")
@@
 	)
 	(segment
-		(start 125.5 80.5)
-		(end 126.95 80.5)
-		(width 1)
-		(layer "B.Cu")
-		(net 3)
-	)
-	(segment
 		(start 130.365831 85.55)
 		(end 128.45 85.55)
@@
 	)
 	(segment
-		(start 123.267084 82.732916)
-		(end 123.267084 83.5)
-		(width 1)
-		(layer "B.Cu")
-		(net 3)
-	)
-	(segment
 		(start 116.635485 91.5)
 		(end 116.635485 90.635485)
@@
 	)
 	(segment
-		(start 127.5 84.6)
-		(end 128.45 85.55)
-		(width 0.5)
-		(layer "B.Cu")
-		(net 3)
-	)
-	(segment
 		(start 116.333063 92.635)
 		(end 117.5 93.801937)
@@
 	)
 	(segment
-		(start 126.95 80.5)
-		(end 131.55 75.9)
-		(width 1)
-		(layer "B.Cu")
-		(net 3)
-	)
-	(segment
 		(start 80.793735 91.5875)
 		(end 80.286235 91.08)
@@
 	)
 	(segment
+		(start 123.95 83.5)
+		(end 123.267084 83.5)
+		(width 1)
+		(layer "B.Cu")
+		(net 3)
+	)
+	(segment
 		(start 90 80.925)
 		(end 91 79.925)
@@
 	)
 	(segment
-		(start 127.5 84.275)
-		(end 127.5 84.6)
-		(width 0.5)
-		(layer "B.Cu")
-		(net 3)
-	)
-	(segment
 		(start 72.5 77)
 		(end 72.5 79.925)
@@
 	)
 	(segment
-		(start 125.317084 85.55)
-		(end 123.267084 83.5)
+		(start 131.55 75.9)
+		(end 123.95 83.5)
 		(width 1)
 		(layer "B.Cu")
@@
 	)
 	(segment
-		(start 125.5 80.5)
-		(end 123.267084 82.732916)
+		(start 125.317084 85.55)
+		(end 123.267084 83.5)
 		(width 1)
 		(layer "B.Cu")
