File: Control Board/Control Board.kicad_pcb (KiCad board)
At the start: 2 copper layers, 89.2 x 84.8 mm, 31 parts, among them J1 Conn_02x14_Odd_Even, J2 I2C 1, J3 I2C 2, J4 SERVO_1, J5 SERVO_3, J6 SERVO_2, J7 SERVO_4, J8 UART 1, J9 UART 2, U1 Teensy4.1

Commit message: Started STM32 based firmware
Connections:
- U2 pad 3: /SDA -> /SCL
- U2 pad 4: /SCL -> /SDA
Routing:
- net /SDA: track 56.0 -> 58.5 mm
- net /SCL: track 63.5 -> 61.6 mm
Other:
- board text added: "Cardinal Control V1.1"
- board text removed: "Cardinal Control V1"
Changed lines of the file:
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@@
 		(allow_soldermask_bridges_in_footprints no)
 		(pcbplotparams
-			(layerselection 0x00010fc_ffffffff)
+			(layerselection 0x0001000_7fffffff)
 			(plot_on_all_layers_selection 0x0000000_00000000)
 			(disableapertmacros no)
@@
 			(psnegative no)
 			(psa4output no)
-			(plotreference yes)
-			(plotvalue yes)
-			(plotfptext yes)
+			(plotreference no)
+			(plotvalue no)
+			(plotfptext no)
 			(plotinvisibletext no)
 			(sketchpadsonfab no)
 			(subtractmaskfromsilk no)
-			(outputformat 1)
+			(outputformat 3)
 			(mirror no)
-			(drillshape 1)
+			(drillshape 2)
 			(scaleselection 1)
 			(outputdirectory "")
@@
 			(layers "*.Cu" "*.Mask")
 			(remove_unused_layers no)
-			(net 13 "/SDA")
+			(net 11 "/SCL")
 			(pinfunction "SCL/SCK/RX")
 			(pintype "input")
@@
 			(layers "*.Cu" "*.Mask")
 			(remove_unused_layers no)
-			(net 11 "/SCL")
+			(net 13 "/SDA")
 			(pinfunction "SDA/MISO/TX")
 			(pintype "output")
@@
 		)
 	)
-	(gr_text "Cardinal\nControl V1"
+	(gr_text "Cardinal\nControl V1.1"
 		(at 116.5 97.5 0)
 		(layer "F.SilkS")
@@
 			(justify left bottom)
 		)
-		(render_cache "Cardinal\nControl V1" 0
+		(render_cache "Cardinal\nControl V1.1" 0
 			(polygon
 				(pts
@@
 				)
 			)
+			(polygon
+				(pts
+					(xy 138.025366 96.99) (xy 138.025366 96.427264) (xy 138.604954 96.427264) (xy 138.604954 96.99)
+				)
+			)
+			(polygon
+				(pts
+					(xy 140.550348 96.99) (xy 139.971493 96.99) (xy 139.971493 94.784487) (xy 139.848523 94.897916)
+					(xy 139.717568 94.999703) (xy 139.578627 95.089845) (xy 139.431701 95.168345) (xy 139.276789 95.235201)
+					(xy 139.223377 95.254898) (xy 139.223377 94.692163) (xy 139.368749 94.634088) (xy 139.506192 94.560041)
+					(xy 139.633618 94.476899) (xy 139.715771 94.416657) (xy 139.838319 94.310594) (xy 139.939986 94.196106)
+					(xy 140.020769 94.07319) (xy 140.080669 93.941849) (xy 140.550348 93.941849)
+				)
+			)
 		)
 	)
@@
 	)
 	(segment
-		(start 93.499998 77.525002)
-		(end 93.499998 78.989998)
+		(start 94.575002 77.525002)
+		(end 93.499998 77.525002)
 		(width 0.2)
 		(layer "B.Cu")
@@
 	)
 	(segment
-		(start 80.069976 65.408505)
-		(end 80.069976 64.336024)
+		(start 99.7 82.65)
+		(end 94.575002 77.525002)
 		(width 0.2)
 		(layer "B.Cu")
@@
 	)
 	(segment
-		(start 62 73.5)
-		(end 63.5 73.5)
+		(start 80.069976 65.408505)
+		(end 80.069976 64.336024)
 		(width 0.2)
 		(layer "B.Cu")
@@
 	)
 	(segment
-		(start 93.499998 78.989998)
-		(end 99.7 85.19)
+		(start 62 73.5)
+		(end 63.5 73.5)
 		(width 0.2)
 		(layer "B.Cu")
@@
 	)
 	(segment
-		(start 93.1574 76.725)
-		(end 81.6892 65.2568)
-		(width 0.2)
-		(layer "F.Cu")
-		(net 13)
-	)
-	(segment
 		(start 81.6892 65.2568)
 		(end 80.7668 65.2568)
@@
 	)
 	(segment
-		(start 93.499998 76.725)
-		(end 93.1574 76.725)
+		(start 93.107622 76.392378)
+		(end 92.824778 76.392378)
 		(width 0.2)
 		(layer "F.Cu")
@@
 	)
 	(segment
+		(start 92.824778 76.392378)
+		(end 81.6892 65.2568)
+		(width 0.2)
+		(layer "F.Cu")
+		(net 13)
+	)
+	(segment
 		(start 64.140365 71.09)
 		(end 66.230365 69)
@@
 	)
 	(via
-		(at 93.499998 76.725)
+		(at 93.107622 76.392378)
 		(size 0.6)
 		(drill 0.3)
@@
 	)
 	(segment
-		(start 93.775 76.725)
-		(end 99.7 82.65)
+		(start 93.107622 76.392378)
+		(end 92.899998 76.600002)
+		(width 0.2)
+		(layer "B.Cu")
+		(net 13)
+	)
+	(segment
+		(start 95 80.49)
+		(end 99.7 85.19)
+		(width 0.2)
+		(layer "B.Cu")
+		(net 13)
+	)
+	(segment
+		(start 95 80)
+		(end 95 80.49)
+		(width 0.2)
+		(layer "B.Cu")
+		(net 13)
+	)
+	(segment
+		(start 92.899998 77.899998)
+		(end 95 80)
 		(width 0.2)
 		(layer "B.Cu")
@@
 	)
 	(segment
-		(start 93.499998 76.725)
-		(end 93.775 76.725)
+		(start 92.899998 76.600002)
+		(end 92.899998 77.899998)
 		(width 0.2)
 		(layer "B.Cu")
