File: Control Board/Control Board.kicad_sch (KiCad schematic)
At the start: 31 parts, among them J1 Conn_02x14_Odd_Even, J2 I2C 1, J3 I2C 2, J4 SERVO_1, J5 SERVO_3, J6 SERVO_2, J7 SERVO_4, J8 UART 1, J9 UART 2, U1 Teensy4.1

Commit message: Started STM32 based firmware
Parts:
- R2, R3, R4, R5, R6, R7: value 4.7k -> 10k
Connections:
- net SCL: now also U2.3 (SCL/SCK/RX); no longer U2.4 (SDA/MISO/TX)
- net SDA: now also U2.4 (SDA/MISO/TX); no longer U2.3 (SCL/SCK/RX)
Changed lines of the file:
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@@
 		)
 	)
+	(label "SCL"
+		(at 123.19 30.48 180)
+		(fields_autoplaced yes)
+		(effects
+			(font
+				(size 1.27 1.27)
+			)
+			(justify right bottom)
+		)
+	)
 	(label "SCL_2"
 		(at 38.1 171.45 180)
@@
 		)
 	)
-	(label "SDA"
-		(at 123.19 30.48 180)
-		(fields_autoplaced yes)
-		(effects
-			(font
-				(size 1.27 1.27)
-			)
-			(justify right bottom)
-		)
-	)
 	(label "S_OX_3"
 		(at 255.27 72.39 0)
@@
 		)
 	)
-	(label "SPEED_1"
-		(at 68.58 25.4 0)
+	(label "SDA"
+		(at 123.19 33.02 180)
 		(fields_autoplaced yes)
 		(effects
@@
 				(size 1.27 1.27)
 			)
-			(justify left bottom)
+			(justify right bottom)
 		)
 	)
-	(label "PWM_4"
-		(at 194.31 44.45 180)
+	(label "SPEED_1"
+		(at 68.58 25.4 0)
 		(fields_autoplaced yes)
 		(effects
@@
 				(size 1.27 1.27)
 			)
-			(justify right bottom)
+			(justify left bottom)
 		)
 	)
-	(label "SCL"
-		(at 123.19 33.02 180)
+	(label "PWM_4"
+		(at 194.31 44.45 180)
 		(fields_autoplaced yes)
 		(effects
@@
 			)
 		)
-		(property "Value" "4.7k"
+		(property "Value" "10k"
 			(at 114.3 162.5599 0)
 			(effects
@@
 			)
 		)
-		(property "Value" "4.7k"
+		(property "Value" "10k"
 			(at 29.21 33.0199 0)
 			(effects
@@
 			)
 		)
-		(property "Value" "4.7k"
+		(property "Value" "10k"
 			(at 54.61 161.2899 0)
 			(effects
@@
 			)
 		)
-		(property "Value" "4.7k"
+		(property "Value" "10k"
 			(at 105.41 162.5599 0)
 			(effects
@@
 			)
 		)
-		(property "Value" "4.7k"
+		(property "Value" "10k"
 			(at 38.1 33.0199 0)
 			(effects
@@
 			)
 		)
-		(property "Value" "4.7k"
+		(property "Value" "10k"
 			(at 45.72 161.2899 0)
 			(effects
